Commit message: update environment

File: model/scene.xml.xacro (robot description, xacro)
@@ -12,12 +12,18 @@
   </extension>
   <asset>
-  <texture name="texchecker" type="2d" builtin="checker" width="512" height="512"
-           rgb1="0.8 0.8 0.8" rgb2="0.2 0.2 0.2" />
-  <material name="matchecker" texture="texchecker" texrepeat="4 4"
-            reflectance="0.2" shininess="0.5" specular="0.3" />
+    <texture name="texwood" type="2d" builtin="gradient" width="512" height="512"
+             rgb1="0.80 0.65 0.45" rgb2="0.65 0.50 0.35" />
+    <material name="matwood" texture="texwood" texrepeat="1 15"
+              reflectance="0.02" shininess="0.05" specular="0.1" />
+    <material name="mat_red"   rgba="0.8 0.1 0.1 1" reflectance="0.01" shininess="0.01" specular="0.0" />
+    <material name="mat_green" rgba="0.1 0.8 0.1 1" reflectance="0.01" shininess="0.01" specular="0.0" />
+    <material name="mat_blue"  rgba="0.1 0.1 0.8 1" reflectance="0.01" shininess="0.01" specular="0.0" />
   </asset>
   <worldbody>
     <light pos="0 0 1.5" dir="0 0 -1" directional="true"/>
-    <geom name="floor" type="plane" size="20 20 0.1" material="matchecker" rgba="1 1 1 1" condim="3"/>
+    <geom name="floor" type="box" pos="2.5 0 -0.05" size="5.5 2 0.05" material="matwood" condim="3"/>
+    <geom name="box_red" type="box" pos="2 1 0.1" size="0.2 0.2 0.1" material="mat_red" />
+    <geom name="box_green" type="box" pos="4 -1 0.1" size="0.2 0.2 0.1" material="mat_green" />
+    <geom name="box_blue" type="box" pos="6 1 0.1" size="0.2 0.2 0.1" material="mat_blue" />
     <xacro:quadrotor_body prefix="quadrotor" pos="0 0 0.02" euler="0 0 0" />
     <body name="payload" pos="1 0 0.02">
@@ -33,4 +39,5 @@
     <geom name="origin_y" type="cylinder" fromto="0 0 0.01 0 0.5 0.01" size="0.01" rgba="0 1 0 0.1" contype="0" conaffinity="0" group="1"/>
     <geom name="origin_z" type="cylinder" fromto="0 0 0.01 0 0 0.51" size="0.01" rgba="0 0 1 0.1" contype="0" conaffinity="0" group="1"/>
+    <camera name="camera_pov" pos="-2.427 1.392 1.622" xyaxes="-0.216 -0.976 -0.000 0.227 -0.050 0.973"/>
   </worldbody>
   <actuator>
@@ -46,8 +53,8 @@
   </sensor>
   <tendon>
-        <spatial name="rope0" limited="true" range="0 1" width=".0005">
-            <site site="quadrotor_payload_site"/>
-            <site site="payload_connection_site"/>
-        </spatial>
+    <spatial name="rope0" limited="true" range="0 1" width=".0005">
+      <site site="quadrotor_payload_site"/>
+      <site site="payload_connection_site"/>
+    </spatial>
   </tendon>
 </mujoco>
